Commit message: publish arm joints to /joint_states and changed xacro

File: spot_description/urdf/spot.urdf.xacro (robot description, xacro)
@@ -259,4 +259,149 @@
         <limit effort="1000" velocity="1000.00" lower="-2.7929" upper="-0.257725" />
     </joint>
+        <!-- Arm addition to XACRO -->
+  <!-- begin arm -->
+  <link name="arm0.link_sh0">
+    <visual>
+      <geometry>
+        <mesh filename="package://spot_description/spot/meshes/arm0_link_sh0.dae"/>
+      </geometry>
+    </visual>
+    <inertial>
+      <origin xyz="-0.008399 0.000272 -0.024603"/>
+      <inertia ixx="0.008896" ixy="0.000005" ixz="-0.000193" iyy="0.004922" iyz="0.000033" izz="0.0073030"/>
+      <mass value="1.904699"/>
+    </inertial>
+  </link>
+  <link name="arm0.link_sh1">
+    <visual>
+      <geometry>
+        <mesh filename="package://spot_description/spot/meshes/arm0_link_sh1.dae"/>
+      </geometry>
+    </visual>
+    <visual>
+      <geometry>
+        <mesh filename="package://spot_description/spot/meshes/arm0_link_hr0.dae"/>
+      </geometry>
+    </visual>
+    <inertial>
+      <origin xyz="0.08084909 -0.00167243 0.00045644"/>
+      <inertia ixx="0.00261526" ixy="-0.00040406" ixz="0.00010019" iyy="0.02703868" iyz="0.00000547" izz="0.02819929"/>
+      <mass value="1.85701942"/>
+    </inertial>
+  </link>
+  <link name="arm0.link_el0">
+    <visual>
+      <geometry>
+        <mesh filename="package://spot_description/spot/meshes/arm0_link_el0.dae"/>
+      </geometry>
+    </visual>
+    <inertial>
+      <origin xyz="0.04476621 -0.00271130 0.04991363"/>
+      <inertia ixx="0.00175909" ixy="0.00006087" ixz="0.00092380" iyy="0.00269233" iyz="0.00005217" izz="0.00202854"/>
+      <mass value="0.94831958"/>
+    </inertial>
+  </link>
+  <link name="arm0.link_el1">
+    <visual>
+      <geometry>
+        <mesh filename="package://spot_description/spot/meshes/arm0_link_el1.dae"/>
+      </geometry>
+    </visual>
+    <inertial>
+      <origin xyz="-0.16867073 -0.01616121 0.00001149"/>
+      <inertia ixx="0.00117710" ixy="-0.00260549" ixz="0.00000156" iyy="0.01649389" iyz="-0.00000287" izz="0.01689901"/>
+      <mass value="1.01754820"/>
+    </inertial>
+  </link>
+  <link name="arm0.link_wr0">
+    <visual>
+      <geometry>
+        <mesh filename="package://spot_description/spot/meshes/arm0_link_wr0.dae"/>
+      </geometry>
+    </visual>
+    <inertial>
+      <origin xyz="0.00952465 -0.01144406 0.00000186"/>
+      <inertia ixx="0.00046738" ixy="0.00006957" ixz="0.00000040" iyy="0.00044968" iyz="0.00000016" izz="0.00053616"/>
+      <mass value="0.58263740"/>
+    </inertial>
+  </link>
+  <link name="arm0.link_wr1">
+    <visual>
+      <geometry>
+        <mesh filename="package://spot_description/spot/meshes/arm0_link_wr1.dae"/>
+      </geometry>
+    </visual>
+    <inertial>
+      <origin xyz="0.09751283 0.00009265 -0.01120523"/>
+      <inertia ixx="0.00098836" ixy="-0.00000126" ixz="-0.00036919" iyy="0.00197018" iyz="-0.00000074" izz="0.00165791"/>
+      <mass value="0.93335298"/>
+    </inertial>
+  </link>
+  <link name="arm0.link_fngr">
+    <visual>
+      <geometry>
+        <mesh filename="package://spot_description/spot/meshes/arm0_link_fngr.dae"/>
+      </geometry>
+    </visual>
+    <inertial>
+      <origin xyz="0.03565178 0.00067200 -0.01227516"/>
+      <inertia ixx="0.00025226" ixy="-0.00000536" ixz="-0.00015067" iyy="0.00048453" iyz="0.00000184" izz="0.00059145"/>
+      <mass value="0.22383315"/>
+    </inertial>
+  </link>
+  <joint name="arm_shoulder_0" type="revolute">
+    <parent link="base_link"/>
+    <child link="arm0.link_sh0"/>
+    <origin xyz="0.292 0.0 0.188"/>
+    <axis xyz="0 0 1"/>
+    <limit effort="90.9" lower="-2.61799" upper="3.14159" velocity="999"/>
+    <dynamics damping="0" friction="10"/>
+  </joint>
+  <joint name="arm_shoulder_1" type="revolute">
+    <parent link="arm0.link_sh0"/>
+    <child link="arm0.link_sh1"/>
+    <origin xyz="0.0 0.0 0.0"/>
+    <axis xyz="0 1 0"/>
+    <limit effort="181.8" lower="-3.14159" upper="0.523599" velocity="999"/>
+    <dynamics damping="0" friction="10"/>
+  </joint>
+  <joint name="arm_elbow_0" type="revolute">
+    <parent link="arm0.link_sh1"/>
+    <child link="arm0.link_el0"/>
+    <origin xyz="0.3385 0 0"/>
+    <axis xyz="0 1 0"/>
+    <limit effort="90.9" lower="0" upper="3.14159" velocity="999"/>
+    <dynamics damping="0" friction="10"/>
+  </joint>
+  <joint name="arm_elbow_1" type="revolute">
+    <parent link="arm0.link_el0"/>
+    <child link="arm0.link_el1"/>
+    <origin xyz="0.40330 0.0 0.0750"/>
+    <axis xyz="1 0 0"/>
+    <limit effort="30.3" lower="-2.792530" upper="2.792530" velocity="999"/>
+    <dynamics damping="0" friction="10"/>
+  </joint>
+  <joint name="arm_wrist_0" type="revolute">
+    <parent link="arm0.link_el1"/>
+    <child link="arm0.link_wr0"/>
+    <axis xyz="0 1 0"/>
+    <limit effort="30.3" lower="-1.8326" upper="1.8326" velocity="999"/>
+    <dynamics damping="0" friction="10"/>
+  </joint>
+  <joint name="arm_wrist_1" type="revolute">
+    <parent link="arm0.link_wr0"/>
+    <child link="arm0.link_wr1"/>
+    <axis xyz="1 0 0"/>
+    <limit effort="30.3" lower="-2.87989" upper="2.87979" velocity="999"/>
+    <dynamics damping="0" friction="10"/>
+  </joint>
+  <joint name="arm_f1x" type="revolute">
+    <parent link="arm0.link_wr1"/>
+    <child link="arm0.link_fngr"/>
+    <origin xyz="0.11745 0 0.014820"/>
+    <axis xyz="0 1 0"/>
+    <limit effort="15.32" lower="-1.5708" upper="0.0" velocity="999"/>
+    <dynamics damping="0" friction="10"/>
+  </joint>
     <!-- Standard accessories. -->
     <xacro:include filename="$(find spot_description)/urdf/accessories.urdf.xacro" />
